File: zephyrus_fc/zephyrus_fc.kicad_sch (KiCad schematic)
At the start: 58 parts, among them J1 SWD_interface, J10 Conn_02x20_Counter_Clockwise, J11 Conn_02x04_Counter_Clockwise, J2 POWER, J3 SERVO1, J4 SERVO2, J5 SERVO3, J6 SERVO4, J7 SERVO5, J8 IBUS_RX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

Commit message: ready to order
Parts:
- added J12: GPS_UART, Connector_PinHeader_2.54mm:PinHeader_1x06_P2.54mm_Vertical, symbol Connector_Generic:Conn_01x06
- added J13: USART2, Connector_PinHeader_2.54mm:PinHeader_1x06_P2.54mm_Vertical, symbol Connector_Generic:Conn_01x06
- added J15, J16: Conn_01x04, Connector_PinHeader_2.54mm:PinHeader_1x04_P2.54mm_Vertical, symbol Connector_Generic:Conn_01x04
- added R11, R12, R13, R14, R7, R8: 2.2k, Resistor_SMD:R_0402_1005Metric, symbol Device:R
Connections:
- net +3.3V: now also R11.1, R12.1, R13.1, R14.1, R7.1, R8.1
- net GND: now also J12.1 (Pin_1), J13.1 (Pin_1), J15.1 (Pin_1), J16.1 (Pin_1)
- net PD3: now also J13.2 (Pin_2)
- net PD4: now also J13.3 (Pin_3)
- net PD5: now also J13.4 (Pin_4)
- net PD6: now also J13.5 (Pin_5)
- net PE0: now also J12.4 (Pin_4)
- net PE1: now also J12.5 (Pin_5)
- net PB10 renamed I2C2_SCL
- net I2C2_SCL: now also J15.3 (Pin_3), R11.2
- net PB11 renamed I2C2_SDA
- net I2C2_SDA: now also J15.2 (Pin_2), R12.2
- net PB8 renamed I2C1_SCL
- net I2C1_SCL: now also J12.3 (Pin_3), R7.2
- net PB9 renamed I2C1_SDA
- net I2C1_SDA: now also J12.2 (Pin_2), R8.2
- net PD12 renamed I2C4_SCL
- net I2C4_SCL: now also J16.3 (Pin_3), R13.2
- net PD13 renamed I2C4_SDA
- net I2C4_SDA: now also J16.2 (Pin_2), R14.2
- net VCC renamed +5V
- net +5V: now also J12.6 (Pin_6), J13.6 (Pin_6), J15.4 (Pin_4), J16.4 (Pin_4)
Other:
- note added: "SENSORS"
- note removed: "USE INTERUPTS"
- moved on the sheet: C1, C10, C11, C12, C13, C14, C15, C16, C17, C18, C19, C2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

Commit message: silkscreened
Parts:
- added J14, J17: POWER, Connector_PinHeader_2.54mm:PinHeader_1x02_P2.54mm_Vertical, symbol Connector_Generic:Conn_01x02
Connections:
- net +5V: now also J14.2 (Pin_2), J17.2 (Pin_2)
- net GND: now also J14.1 (Pin_1), J17.1 (Pin_1)
